File: fpgaboard.kicad_sch (KiCad schematic)
At the start: 20 parts, among them J1 Conn_02x06_Odd_Even, J2 Conn_02x06_Odd_Even, J3 Conn_02x06_Odd_Even, J4 Conn_02x06_Odd_Even, J5 Conn_02x06_Odd_Even, J6 Conn_02x06_Odd_Even, J7 Conn_02x20_Odd_Even, SW1 SW_Push, SW2 SW_Push, U1 ICE40HX4K-TQ144

Commit message: flash added
Parts:
- added C2: 100n, symbol Device:C
- added R8, R9: R, symbol Device:R
- added is25lp016d-jble1: ~, symbol is25lp016d-jble:is25lp016d-jble_
Connections:
- net +3.3V: now also C2.1, is25lp016d-jble1. (VCC)
- net GND: now also C2.2, is25lp016d-jble1. (VCC)
- net gp10: now also is25lp016d-jble1. (VCC)
- net gp11: now also is25lp016d-jble1. (VCC)
- net gp8: now also is25lp016d-jble1. (VCC)
- net gp9: now also is25lp016d-jble1. (VCC)
- net sd_io2: now also is25lp016d-jble1. (VCC)
- net sd_io3: now also is25lp016d-jble1. (VCC)
- new net +3V3: R8.1, R9.1
- new net sd1o2: R9.2
- new net sd1o3: R8.2
Other:
- note added: "FLASH"
- note added: "Rest of the fpga pins are added above"

Commit message: fpgaboard
Parts:
- added C10, C11, C12, C13, C14, C15, C16, C17, C18, C19, C20, C3, C8, C9: 100n, symbol Device:C
- added C4, C5, C6, C7: 1u, symbol Device:C
- added G1: SiT2001BI-S2-33E-12.000000, SiT2001BI-S2-33E-12.000000:SOT95P280X145-5N, symbol clock12mhz:SiT2001BI-S2-33E-12.000000
- added L1, L2, L3: L, symbol Device:L
- added U2: TLV73312PDBV, Package_TO_SOT_SMD:SOT-23-5, symbol Regulator_Linear:TLV73312PDBV
- added U3: TLV73333PDBV, Package_TO_SOT_SMD:SOT-23-5, symbol Regulator_Linear:TLV73333PDBV
Connections:
- net +3.3V: now also C12.1, C13.1, C14.1, C15.1, C16.1, C17.1, C18.1, C19.1, C20.1, C3.1, G1.3 (OE), G1.4 (VDD), L2.2, L3.1, L3.2
- net +5V: now also C4.1, C6.1, U2.1 (IN), U2.3 (EN), U3.1 (IN), U3.3 (EN)
- net GND: now also C10.2, C11.2, C12.2, C13.2, C14.2, C15.2, C16.2, C17.2, C18.2, C19.2, C20.2, C3.2, C4.2, C5.2, C6.2, C7.2, C8.2, C9.2, G1.1 (GND), U2.2 (GND), U3.2 (GND)
- net clock: now also G1.5 (OUT)
- new net: C7.1, L2.1, U3.5 (OUT)
- new net: C5.1, L1.1, U2.5 (OUT)
- new net +1V2: C10.1, C11.1, C8.1, C9.1, L1.2
Other:
- note added: "CLOCK"
- note added: "POWER SUPPLY"
- note added: "PROGRAMMING"
- moved on the sheet: C2, R8, R9, is25lp016d-jble1

Commit message: fpgaboard
Parts:
- C1, C10, C11, C12, C13, C14, C15, C16, C17, C18, C19, C2, C20, C3, C4, C5, C6, C7, C8, C9: footprint (none) -> Capacitor_SMD:C_0201_0603Metric_Pad0.64x0.40mm_HandSolder
- D1, D2: footprint (none) -> LED_SMD:LED_0201_0603Metric_Pad0.64x0.40mm_HandSolder
- G1: footprint SiT2001BI-S2-33E-12.000000:SOT95P280X145-5N -> clock12Mhz:SOT95P280X145-5N
- J1, J2, J3, J4, J5, J6: footprint (none) -> Connector_PinSocket_2.54mm:PinSocket_2x06_P2.54mm_Horizontal
- J7: footprint (none) -> Connector_PinSocket_2.54mm:PinSocket_2x20_P2.54mm_Horizontal
- L1, L2, L3: footprint (none) -> Inductor_SMD:L_0201_0603Metric_Pad0.64x0.40mm_HandSolder
- R1, R2, R3, R4, R5, R6, R7, R8, R9: footprint (none) -> Resistor_SMD:R_0201_0603Metric_Pad0.64x0.40mm_HandSolder

Commit message: fpgaboard
Parts:
- SW1, SW2: footprint (none) -> Button_Switch_THT:SW_DIP_SPSTx01_Slide_6.7x4.1mm_W7.62mm_P2.54mm_LowProfile
- is25lp016d-jble1: footprint (none) -> flash:SOIC127P790X216-8N
Connections:
- net sd1o2 is gone; now on net sd_io2: R9.2
- net sd1o3 is gone; now on net sd_io3: R8.2
- net +3.3V: now also is25lp016d-jble1.8 (VCC); no longer is25lp016d-jble1. (VCC)
- net GND: now also is25lp016d-jble1.4 (GND); no longer is25lp016d-jble1. (VCC)
- net cdone: now also J7.31 (Pin_31); no longer J7.11 (Pin_11)
- net creset: now also J7.33 (Pin_33); no longer J7.13 (Pin_13)
- net gp0: now also J7.38 (Pin_38); no longer J7.27 (Pin_27)
- net gp10: now also is25lp016d-jble1.5 (D1(IO0)); no longer is25lp016d-jble1. (VCC)
- net gp11: now also is25lp016d-jble1.6 (CLK); no longer is25lp016d-jble1. (VCC)
- net gp12: now also J7.15 (Pin_15); no longer J7.32 (Pin_32)
- net gp13: now also J7.13 (Pin_13); no longer J7.33 (Pin_33)
- net gp16: now also J7.11 (Pin_11); no longer J7.36 (Pin_36)
- net gp20: now also J7.5 (Pin_5); no longer J7.38 (Pin_38)
- net gp21: now also J7.7 (Pin_7); no longer J7.40 (Pin_40)
- net gp22: now also J7.32 (Pin_32); no longer J7.15 (Pin_15)
- net gp3: now also J7.27 (Pin_27); no longer J7.5 (Pin_5)
- net gp4: now also J7.29 (Pin_29); no longer J7.7 (Pin_7)
- net gp5: now also J7.40 (Pin_40); no longer J7.29 (Pin_29)
- net gp6: now also J7.17 (Pin_17); no longer J7.31 (Pin_31)
- net gp8: now also is25lp016d-jble1.1 (CS_bar); no longer is25lp016d-jble1. (VCC)
- net gp9: now also is25lp016d-jble1.2 (D0(IO1)); no longer is25lp016d-jble1. (VCC)
- net p1_1: now also J1.12 (Pin_12); no longer J1.11 (Pin_11)
- net p1_10: now also J1.5 (Pin_5); no longer J1.6 (Pin_6)
- net p1_2: now also J1.10 (Pin_10); no longer J1.9 (Pin_9)
- net p1_3: now also J1.8 (Pin_8); no longer J1.7 (Pin_7)
- net p1_4: now also J1.6 (Pin_6); no longer J1.5 (Pin_5)
- net p1_7: now also J1.11 (Pin_11); no longer J1.12 (Pin_12)
- net p1_8: now also J1.9 (Pin_9); no longer J1.10 (Pin_10)
- net p1_9: now also J1.7 (Pin_7); no longer J1.8 (Pin_8)
- net pi_3v3_2: now also J7.36 (Pin_36); no longer J7.17 (Pin_17)
- net sd_io2: now also is25lp016d-jble1.3 (IO2); no longer is25lp016d-jble1. (VCC)
- net sd_io3: now also is25lp016d-jble1.7 (IO3); no longer is25lp016d-jble1. (VCC)
